File: blinken_lights.kicad_pcb (KiCad board)
At the start: 2 copper layers, 31 parts, among them J1 tx, J2 rx, J4 ICSP, SW1 reset, U3 ATtiny841-SSU, U4 LIGHTSENSORTEMT6000

Commit message: major work
done?
art needed
Parts:
- removed J2: rx, TestPoint:TestPoint_Pad_D2.0mm
- removed J4: ICSP, Connector_PinHeader_1.27mm:PinHeader_2x03_P1.27mm_Vertical
- removed JP1, JP2, JP3, JP4, JP5, JP6: JUMPER-2PTH, Connector_PinHeader_1.27mm:PinHeader_1x02_P1.27mm_Vertical
- removed R10: 220, Resistor_SMD:R_0805_2012Metric_Pad1.15x1.40mm_HandSolder
- removed R5, R7, R8: 470, Resistor_SMD:R_0805_2012Metric_Pad1.15x1.40mm_HandSolder
- removed R9: 10k, Resistor_SMD:R_0805_2012Metric_Pad1.15x1.40mm_HandSolder
- removed SW1: reset, Button_Switch_SMD:SW_Push_1P1T_NO_CK_KMR2
- removed U3: ATtiny841-SSU, Package_SO:SOIC-14_3.9x8.7mm_P1.27mm
- removed U4: LIGHTSENSORTEMT6000, SparkFun-Sensors:TEMT6000-SEN
- added C1: C_Small, Resistor_SMD:R_0805_2012Metric_Pad1.15x1.40mm_HandSolder, F.Cu at (222.0, 150.9)
- added G***: LOGO, LOGO, B.Cu at (224.5, 152.9)
- added R1: 470, Resistor_SMD:R_0805_2012Metric_Pad1.15x1.40mm_HandSolder, F.Cu at (211.8, 147.3)
- added R2: 470, Resistor_SMD:R_0805_2012Metric_Pad1.15x1.40mm_HandSolder, F.Cu at (215.4, 147.3)
- added R3: 470, Resistor_SMD:R_0805_2012Metric_Pad1.15x1.40mm_HandSolder, F.Cu at (220.5, 147.3)
- added U1: ATtiny85-20SU, Package_SO:SOIJ-8_5.3x5.3mm_P1.27mm, F.Cu at (217.9, 154.9)
- added VCC1: Conn_01x01_Female, Connector_Pin:Pin_D1.0mm_L10.0mm_LooseFit, F.Cu at (217.9, 150.4)
- J1: value tx -> Conn_01x01_Female; footprint TestPoint:TestPoint_Pad_D2.0mm -> Connector_Pin:Pin_D1.0mm_L10.0mm_LooseFit
- R4: value 10k -> 470
- R6: value 470 -> 10k
- moved J1 27.0 mm to (217.9, 130.6)
- moved R4 6.10 mm to (224.0, 147.3), turned to 225 degrees
- moved R6 5.57 mm to (213.9, 150.9), turned to 0 degrees
- moved D7 3.30 mm to (211.6, 143.3)
- moved D12 3.14 mm to (223.8, 143.3)
- moved D11 2.91 mm to (215.6, 143.3)
- moved D15 2.87 mm to (211.6, 138.7)
- moved D8 2.85 mm to (219.7, 143.3)
- moved D10 2.69 mm to (223.8, 138.7)
- moved D5 2.48 mm to (211.6, 134.1)
- moved D16 2.42 mm to (215.6, 138.7)
- moved D6 2.35 mm to (219.7, 138.7)
- moved D14 2.27 mm to (223.8, 134.1)
- moved D9 1.94 mm to (215.6, 134.1)
- moved D13 1.85 mm to (219.7, 134.1)
Connections:
- D10 pad 1: (no net) -> Net-(D10-Pad1)
- D10 pad 2: (no net) -> Net-(D10-Pad2)
- D11 pad 1: (no net) -> Net-(D10-Pad2)
- D11 pad 2: (no net) -> Net-(D11-Pad2)
- D12 pad 1: (no net) -> Net-(D10-Pad1)
- D12 pad 2: (no net) -> Net-(D11-Pad2)
- D13 pad 1: (no net) -> Net-(D10-Pad2)
- D13 pad 2: (no net) -> Net-(D13-Pad2)
- D14 pad 1: (no net) -> Net-(D13-Pad2)
- D14 pad 2: (no net) -> Net-(D10-Pad2)
- D15 pad 1: (no net) -> Net-(D11-Pad2)
- D15 pad 2: (no net) -> Net-(D13-Pad2)
- D16 pad 1: (no net) -> Net-(D13-Pad2)
- D16 pad 2: (no net) -> Net-(D11-Pad2)
- D5 pad 1: (no net) -> Net-(D10-Pad1)
- D5 pad 2: (no net) -> Net-(D13-Pad2)
- D6 pad 1: (no net) -> Net-(D10-Pad2)
- D6 pad 2: (no net) -> Net-(D10-Pad1)
- D7 pad 1: (no net) -> Net-(D11-Pad2)
- D7 pad 2: (no net) -> Net-(D10-Pad2)
- D8 pad 1: (no net) -> Net-(D11-Pad2)
- D8 pad 2: (no net) -> Net-(D10-Pad1)
- D9 pad 1: (no net) -> Net-(D13-Pad2)
- D9 pad 2: (no net) -> Net-(D10-Pad1)
- J1 pad 1: (no net) -> Earth
- R4 pad 1: (no net) -> Net-(D11-Pad2)
- R4 pad 2: (no net) -> /charlie_leds/in_3
- R6 pad 1: (no net) -> Net-(R6-Pad1)
- R6 pad 2: (no net) -> +3V0
Routing:
- net (no net): track 614.6 -> 0.00 mm, vias 24 -> 0
- net Net-(D13-Pad2): track 0.00 -> 38.6 mm
- net Net-(D10-Pad1): track 0.00 -> 37.4 mm, vias 0 -> 3
- net Net-(D10-Pad2): track 0.00 -> 31.0 mm, vias 0 -> 2
- net Net-(D11-Pad2): track 0.00 -> 24.1 mm
- net /charlie_leds/in_1: track 0.00 -> 15.1 mm, vias 0 -> 2
- net /charlie_leds/in_2: track 0.00 -> 13.0 mm, vias 0 -> 2
- net /charlie_leds/in_4: track 0.00 -> 10.6 mm, vias 0 -> 2
- net /charlie_leds/in_3: track 0.00 -> 10.2 mm, vias 0 -> 2
- net +3V0: track 0.00 -> 8.92 mm
- net Earth: track 0.00 -> 7.06 mm, vias 0 -> 3
- net Net-(R6-Pad1): track 0.00 -> 3.55 mm
- added copper zone on F.Cu, net (none)
- added copper zone on B.Cu, net Earth
Other:
- board outline added: 21.3 x 30.5 mm
