File: charlie.sch (KiCad schematic (older format))
At the start: 16 parts

Commit message: major work
done?
art needed
Parts:
- renumbered D6 to D10, D7 to D11, D8 to D12, D9 to D13, D10 to D14, D11 to D15, D12 to D16, D1 to D5, D2 to D6, D3 to D7, D4 to D8, D5 to D9
Changed lines of the file:
@@
 $Descr A4 11693 8268
 encoding utf-8
-Sheet 2 3
+Sheet 2 2
 Title ""
 Date ""
@@
 $EndComp
 $Comp
-L Device:LED D1
+L Device:LED D5
 U 1 1 5D2C5052
 P 4800 2550
-F 0 "D1" V 4839 2433 50  0000 R CNN
+F 0 "D5" V 4839 2433 50  0000 R CNN
 F 1 "LED" V 4748 2433 50  0000 R CNN
 F 2 "Diode_SMD:D_0805_2012Metric_Pad1.15x1.40mm_HandSolder" H 4800 2550 50  0001 C CNN
@@
 $EndComp
 $Comp
-L Device:LED D5
+L Device:LED D9
 U 1 1 5D2C5CCD
 P 5150 2550
-F 0 "D5" V 5097 2628 50  0000 L CNN
+F 0 "D9" V 5097 2628 50  0000 L CNN
 F 1 "LED" V 5188 2628 50  0000 L CNN
 F 2 "Diode_SMD:D_0805_2012Metric_Pad1.15x1.40mm_HandSolder" H 5150 2550 50  0001 C CNN
@@
 Connection ~ 4800 2700
 $Comp
-L Device:LED D9
+L Device:LED D13
 U 1 1 5D2CA571
 P 5450 2550
-F 0 "D9" V 5489 2432 50  0000 R CNN
+F 0 "D13" V 5489 2432 50  0000 R CNN
 F 1 "LED" V 5398 2432 50  0000 R CNN
 F 2 "Diode_SMD:D_0805_2012Metric_Pad1.15x1.40mm_HandSolder" H 5450 2550 50  0001 C CNN
@@
 $EndComp
 $Comp
-L Device:LED D10
+L Device:LED D14
 U 1 1 5D2CA577
 P 5800 2550
-F 0 "D10" V 5747 2629 50  0000 L CNN
+F 0 "D14" V 5747 2629 50  0000 L CNN
 F 1 "LED" V 5838 2629 50  0000 L CNN
 F 2 "Diode_SMD:D_0805_2012Metric_Pad1.15x1.40mm_HandSolder" H 5800 2550 50  0001 C CNN
@@
 Connection ~ 5450 3000
 $Comp
-L Device:LED D11
+L Device:LED D15
 U 1 1 5D2CBDF0
 P 6100 2550
-F 0 "D11" V 6139 2432 50  0000 R CNN
+F 0 "D15" V 6139 2432 50  0000 R CNN
 F 1 "LED" V 6048 2432 50  0000 R CNN
 F 2 "Diode_SMD:D_0805_2012Metric_Pad1.15x1.40mm_HandSolder" H 6100 2550 50  0001 C CNN
@@
 $EndComp
 $Comp
-L Device:LED D12
+L Device:LED D16
 U 1 1 5D2CBDF6
 P 6450 2550
-F 0 "D12" V 6397 2629 50  0000 L CNN
+F 0 "D16" V 6397 2629 50  0000 L CNN
 F 1 "LED" V 6488 2629 50  0000 L CNN
 F 2 "Diode_SMD:D_0805_2012Metric_Pad1.15x1.40mm_HandSolder" H 6450 2550 50  0001 C CNN
@@
 Connection ~ 6100 3300
 $Comp
-L Device:LED D2
+L Device:LED D6
 U 1 1 5D2CE956
 P 4800 2850
-F 0 "D2" V 4839 2733 50  0000 R CNN
+F 0 "D6" V 4839 2733 50  0000 R CNN
 F 1 "LED" V 4748 2733 50  0000 R CNN
 F 2 "Diode_SMD:D_0805_2012Metric_Pad1.15x1.40mm_HandSolder" H 4800 2850 50  0001 C CNN
@@
 $EndComp
 $Comp
-L Device:LED D6
+L Device:LED D10
 U 1 1 5D2CE95C
 P 5150 2850
-F 0 "D6" V 5097 2929 50  0000 L CNN
+F 0 "D10" V 5097 2929 50  0000 L CNN
 F 1 "LED" V 5188 2929 50  0000 L CNN
 F 2 "Diode_SMD:D_0805_2012Metric_Pad1.15x1.40mm_HandSolder" H 5150 2850 50  0001 C CNN
@@
 	4800 3000 5450 3000
 $Comp
-L Device:LED D3
+L Device:LED D7
 U 1 1 5D2CF7D3
 P 4800 3150
-F 0 "D3" V 4839 3033 50  0000 R CNN
+F 0 "D7" V 4839 3033 50  0000 R CNN
 F 1 "LED" V 4748 3033 50  0000 R CNN
 F 2 "Diode_SMD:D_0805_2012Metric_Pad1.15x1.40mm_HandSolder" H 4800 3150 50  0001 C CNN
@@
 $EndComp
 $Comp
-L Device:LED D7
+L Device:LED D11
 U 1 1 5D2CF7D9
 P 5150 3150
-F 0 "D7" V 5097 3229 50  0000 L CNN
+F 0 "D11" V 5097 3229 50  0000 L CNN
 F 1 "LED" V 5188 3229 50  0000 L CNN
 F 2 "Diode_SMD:D_0805_2012Metric_Pad1.15x1.40mm_HandSolder" H 5150 3150 50  0001 C CNN
@@
 	4800 3300 6100 3300
 $Comp
-L Device:LED D4
+L Device:LED D8
 U 1 1 5D2D2495
 P 4800 3600
-F 0 "D4" V 4839 3483 50  0000 R CNN
+F 0 "D8" V 4839 3483 50  0000 R CNN
 F 1 "LED" V 4748 3483 50  0000 R CNN
 F 2 "Diode_SMD:D_0805_2012Metric_Pad1.15x1.40mm_HandSolder" H 4800 3600 50  0001 C CNN
@@
 	0    -1   -1   0
 $EndComp
-$Comp
-L Device:LED D8
+Wire Wire Line
+	4800 3450 5150 3450
+Wire Wire Line
+	4800 3750 5150 3750
+Wire Wire Line
+	4650 2700 4650 3450
+Connection ~ 4650 2700
+Wire Wire Line
+	4650 2700 4800 2700
+Connection ~ 4800 3450
+Wire Wire Line
+	4600 3300 4600 3750
+Connection ~ 4600 3300
+Wire Wire Line
+	4600 3300 4800 3300
+Connection ~ 4800 3750
+Wire Wire Line
+	4600 3750 4800 3750
+Wire Wire Line
+	4650 3450 4800 3450
+$Comp
+L Device:LED D12
 U 1 1 5D2D249B
 P 5150 3600
-F 0 "D8" V 5097 3679 50  0000 L CNN
+F 0 "D12" V 5097 3679 50  0000 L CNN
 F 1 "LED" V 5188 3679 50  0000 L CNN
 F 2 "Diode_SMD:D_0805_2012Metric_Pad1.15x1.40mm_HandSolder" H 5150 3600 50  0001 C CNN
@@
 	0    1    1    0
 $EndComp
-Wire Wire Line
-	4800 3450 5150 3450
-Wire Wire Line
-	4800 3750 5150 3750
-Wire Wire Line
-	4650 2700 4650 3450
-Connection ~ 4650 2700
-Wire Wire Line
-	4650 2700 4800 2700
-Connection ~ 4800 3450
-Wire Wire Line
-	4600 3300 4600 3750
-Connection ~ 4600 3300
-Wire Wire Line
-	4600 3300 4800 3300
-Connection ~ 4800 3750
-Wire Wire Line
-	4600 3750 4800 3750
-Wire Wire Line
-	4650 3450 4800 3450
 $EndSCHEMATC
